Commit message: rev E updates

File: mh5_description/urdf/mh5_leg_revE.xacro (robot description, xacro)
@@ -253,4 +253,10 @@
             </inertial>
         </link>
+        <joint name="${side}_sole_fixed" type="fixed">
+            <parent link="${side}_foot"/>
+            <child link="${side}_landing"/>
+            <origin xyz="0.0 0.0 -0.03825" rpy="0 0 0"/>
+        </joint>
+        <link name="${side}_landing" />
     </xacro:macro>
 </robot>

File: mh5_description/urdf/mh5_transmission.xacro (robot description, xacro)
@@ -8,5 +8,5 @@
       </joint>
       <actuator name="${name}_motor">
-        <hardwareInterface>hardware_interface/PositionJointInterface</hardwareInterface>
+        <!-- <hardwareInterface>hardware_interface/PositionJointInterface</hardwareInterface> -->
         <mechanicalReduction>1</mechanicalReduction>
       </actuator>
